File: pcb/hackxpansion.kicad_pcb (KiCad board)
At the start: 2 copper layers, 35 parts, among them IC1 ADS7128IRTET, J1 Conn_01x03_MountingPin, J3 Conn_02x07_Counter_Clockwise, J4 Conn_02x07_Counter_Clockwise, J5 Conn_02x07_Counter_Clockwise, J6 Conn_02x07_Counter_Clockwise, Q1 SS8050, SW1 SW_Push, SW2 SW_Push, U2 RP2354B, Y1 ABM8-272-T3

Commit message: worked on power
Parts:
- removed J5, J6: Conn_02x07_Counter_Clockwise, Connector_PinSocket_2.54mm:PinSocket_2x07_P2.54mm_Horizontal
- added C88: 4u7, Capacitor_SMD:C_0402_1005Metric, F.Cu at (160.9, 24.5)
- added C90: 4u7, Capacitor_SMD:C_0402_1005Metric, F.Cu at (160.9, 26.5)
- added C92: 4u7, Capacitor_SMD:C_0402_1005Metric, F.Cu at (160.9, 28.4)
- added C93: 4u7, Capacitor_SMD:C_0402_1005Metric, F.Cu at (160.9, 30.4)
- added Q2: 2N7002, Package_TO_SOT_SMD:SOT-23, F.Cu at (159.3, 33.7)
- added R16: 100k, Resistor_SMD:R_0805_2012Metric, F.Cu at (159.0, 37.4)
- added R28: 3k9, Resistor_SMD:R_0402_1005Metric, F.Cu at (158.0, 24.5)
- added R30: 1k5, Resistor_SMD:R_0402_1005Metric, F.Cu at (158.0, 26.5)
- added R34: 10k, Resistor_SMD:R_0402_1005Metric, F.Cu at (158.0, 28.5)
- added R35: 10k, Resistor_SMD:R_0402_1005Metric, F.Cu at (158.0, 30.5)
- added SW25: SW_On_Off, Button_Switch_THT:SW_CK_JS202011AQN_DPDT_Angled, F.Cu at (148.8, 25.0)
- added U1: ~, Connector_PinSocket_2.54mm:PinSocket_2x07_P2.54mm_Horizontal, F.Cu at (159.6, 43.2)
- added U12: BQ24075RGT, Package_DFN_QFN:VQFN-16-1EP_3x3mm_P0.5mm_EP1.6x1.6mm, F.Cu at (149.0, 34.2)
- added U3: ~, Connector_PinSocket_2.54mm:PinSocket_2x07_P2.54mm_Horizontal, F.Cu at (177.5, 43.2)
- added U4: ~, Connector_PinSocket_2.54mm:PinSocket_2x07_P2.54mm_Horizontal, F.Cu at (177.5, 65.0)
- added U5: ~, Connector_PinSocket_2.54mm:PinSocket_2x07_P2.54mm_Horizontal, F.Cu at (159.6, 65.0)
- added U7: SPX3819M5-L-3-3, Package_TO_SOT_SMD:SOT-23-5, F.Cu at (154.3, 33.9)
- added USB1: TYPE-C 16PIN 2MD, easyeda2kicad:USB-C-SMD_TYPE-C-16PIN-2MD-073, F.Cu at (231.4, 96.2)
- C15, C16: footprint RP2350_80QFN_minimal:C_0402_1005Metric_small_pads -> RP2354B_MINIMAL:C_0402_1005Metric_small_pads
- J3: value Conn_02x07_Counter_Clockwise -> USB_C_Receptacle_USB2.0_14P; footprint Connector_PinSocket_2.54mm:PinSocket_2x07_P2.54mm_Horizontal -> easyeda2kicad:USB-C-SMD_TYPE-C-16PIN-2MD-073
- J4: value Conn_02x07_Counter_Clockwise -> USB_C_Receptacle_USB2.0_14P; footprint Connector_PinSocket_2.54mm:PinSocket_2x07_P2.54mm_Horizontal -> Connector_USB:USB_C_Receptacle_G-Switch_GT-USB-7010ASV
- L1: footprint RP2350_80QFN_minimal:L_pol_2016 -> RP2354B_MINIMAL:L_pol_2016
- Q1: value SS8050 -> BSS138; footprint Package_TO_SOT_THT:TO-92 -> Package_TO_SOT_SMD:SOT-23
- U2: footprint RP2350_80QFN_minimal:RP2350-QFN-80-1EP_10x10_P0.4mm_EP3.4x3.4mm_ThermalVias -> RP2354B_MINIMAL:RP2350-QFN-80-1EP_10x10_P0.4mm_EP3.4x3.4mm_ThermalVias
- moved Q1 114.7 mm to (166.8, 25.7)
- moved J4 60.2 mm to (244.8, 88.9)
- moved J3 48.4 mm to (245.0, 96.3)
Connections:
- net /RP2354B/USB_D+ renamed /RP2354B/D+
- net /RP2354B/USB_D- renamed /RP2354B/D-
- J3 pad 13: unconnected-(J3-Pin_13-Pad13) -> (no net)
- J3 pad 14: unconnected-(J3-Pin_14-Pad14) -> (no net)
- Q1 pad 1: unconnected-(Q1-B-Pad1) -> /Display/BACKLIGHT
- Q1 pad 2: unconnected-(Q1-E-Pad2) -> GND
- Q1 pad 3: unconnected-(Q1-C-Pad3) -> Net-(Q1-D)
