File: pcbs/main_and_daughter/daughter.kicad_sch (KiCad schematic)
At the start: 4 parts

Commit message: added titles to schematic
Other:
- title: (none) -> Daughter Board
Changed lines of the file:
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@@
 	(generator_version "10.0")
 	(paper "A5")
+	(title_block
+		(title "Daughter Board")
+	)
 	(wire
 		(pts
