File: pcbs/main_and_daughter/daughter_conn.kicad_sch (KiCad schematic)
At the start: 1 part, among them CN1 533981471

Commit message: added titles to schematic
Other:
- title: (none) -> Interconnect Connector
Changed lines of the file:
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@@
 	(generator_version "10.0")
 	(paper "A5")
+	(title_block
+		(title "Interconnect Connector")
+	)
 	(junction
 		(at 161.29 91.44)

Commit message: added lcsc part nums
Parts:
- CN1: LCSC (none) -> C2886291; LCSC Part C2886291 -> (none)
Changed lines of the file:
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@@
 			)
 		)
-		(property "LCSC Part" "C2886291"
+		(property "LCSC" "C2886291"
 			(at 157.48 107.95 0)
 			(hide yes)
