File: hardware/hackxpansion/pcb/disp.kicad_sch (KiCad schematic)
At the start: 10 parts, among them Q1 BSS138

Commit message: changed out fpc connector, fixed usb dp width
Parts:
- FPC1: footprint easyeda2kicad:FPC-SMD_AFC08-S12ECA-00 -> easyeda2kicad:FPC-SMD_P0.80-12P_LCS-SJ-H2.0
Changed lines of the file:
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@@
 			)
 		)
-		(property "Footprint" "easyeda2kicad:FPC-SMD_AFC08-S12ECA-00"
+		(property "Footprint" "easyeda2kicad:FPC-SMD_P0.80-12P_LCS-SJ-H2.0"
 			(at 135.89 92.71 0)
 			(hide yes)

Commit message: updated part numbers
Parts:
- FPC1: LCSC C262703 -> C262331
Changed lines of the file:
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@@
 			)
 		)
-		(property "LCSC" "C262703"
+		(property "LCSC" "C262331"
 			(at 135.89 66.04 0)
 			(hide yes)

Commit message: updated module detect resistor to 0.1%
Parts:
- R8: LCSC C2906861 -> C190095
Changed lines of the file:
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@@
 			)
 		)
-		(property "LCSC" "C2906861"
+		(property "LCSC" "C190095"
 			(at 83.82 48.26 0)
 			(hide yes)
