File: hardware/modules/two_button/pcb/two_button.kicad_pcb (KiCad board)
At the start: 2 copper layers, 25.5 x 32 mm, 7 parts, among them SW1 SW_Push, SW2 SW_Push

Commit message: added resistor values to the four and two button modules
Parts:
- R1: value R -> 1k5
- R2: value R -> 1k6
Changed lines of the file:
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@@
 		(capping no)
 		(filling no)
-		(zone_defaults)
 		(grid_origin 132.98 93.72)
 		(pcbplotparams
@@
 			)
 		)
-		(property "Value" "R"
+		(property "Value" "1k5"
 			(at 0 1.65 90)
 			(layer "F.Fab")
@@
 			(at 0 0 90)
 			(layer "F.SilkS")
+			(hide yes)
+			(effects
+				(font
+					(size 1 1)
+					(thickness 0.15)
+				)
+			)
+		)
+		(property "LCSC" "C281775"
+			(at 0 0 270)
+			(unlocked yes)
+			(layer "F.Fab")
 			(hide yes)
 			(effects
@@
 			)
 		)
-		(property "Value" "R"
+		(property "Value" "1k6"
 			(at 0 1.65 0)
 			(layer "F.Fab")
@@
 			(hide yes)
 			(effects
+				(font
+					(size 1 1)
+					(thickness 0.15)
+				)
+			)
+		)
+		(property "LCSC" "C861205"
+			(at 0 0 0)
+			(unlocked yes)
+			(layer "F.Fab")
+			(hide yes)
+			(effects
