File: hardware/modules/hdmi/hdmi/hdmi.kicad_pcb (KiCad board)
At the start: 2 copper layers, 52 x 34.5 mm, 46 parts, among them J1 HDMI_A, U1 BT817Q-T, U2 TFP410PAP, U3 MT25QLxxxxxx1xSE, U4 UCL0524P, U5 UCL0524P, U6 UCL0524P, Y1 12MHz

Commit message: test routing hdmi module
Parts:
- moved U1 1.15 mm to (146.8, 113.8)
- moved J3 1.02 mm to (171.4, 122.8)
- moved U2 0.60 mm to (165.8, 113.8)
- moved U4 0.60 mm to (163.5, 105.9)
- moved U5 0.60 mm to (166.5, 105.9)
- moved J2 0.52 mm to (144.4, 122.8)
Routing:
- net /RGB-HDMI/RGB9: track 0.00 -> 12.7 mm, vias 0 -> 2
- net /RGB-HDMI/RGB15: track 0.00 -> 12.5 mm, vias 0 -> 1
- net /RGB-HDMI/RGB1: track 0.00 -> 12.4 mm, vias 0 -> 2
- net /RGB-HDMI/RGB5: track 0.00 -> 12.4 mm, vias 0 -> 2
- net /RGB-HDMI/RGB2: track 0.00 -> 12.4 mm, vias 0 -> 2
- net /RGB-HDMI/RGB3: track 0.00 -> 12.4 mm, vias 0 -> 2
- net /RGB-HDMI/RGB4: track 0.00 -> 12.4 mm, vias 0 -> 2
- net /RGB-HDMI/RGB11: track 0.00 -> 12.4 mm, vias 0 -> 2
- net /RGB-HDMI/RGB7: track 0.00 -> 11.4 mm, vias 0 -> 2
- net /RGB-HDMI/RGB6: track 0.00 -> 11.4 mm, vias 0 -> 2
- net /RGB-HDMI/RGB13: track 0.00 -> 11.3 mm, vias 0 -> 1
- net /RGB-HDMI/RGB8: track 0.00 -> 11.1 mm, vias 0 -> 2
- net /RGB-HDMI/RGB14: track 0.00 -> 11.1 mm, vias 0 -> 1
- net /RGB-HDMI/RGB10: track 0.00 -> 11.0 mm, vias 0 -> 2
- net /RGB-HDMI/RGB0: track 0.00 -> 10.8 mm, vias 0 -> 2
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